Commit message: update new urdf

File: legged_gym/resources/robots/sirius/urdf/sirius_diff.urdf (robot description, URDF)
Before this commit: robot robot, 18 links, 17 joints
Joints:
- joint LF_HAA: limit lower=-0.7853981633974483 upper=0.7853981633974483 effort=35 velocity=10 -> lower=-0.7853981633974483 upper=0.7853981633974483 effort=40 velocity=10
- joint LF_HFE: limit lower=-1.57 upper=2.5 effort=35 velocity=10 -> lower=-1.57 upper=2.5 effort=40 velocity=10
- joint LF_KFE: limit lower=-3.141592653589793 upper=1.17453292519943295 effort=45 velocity=10 -> lower=-3.141592653589793 upper=1.17453292519943295 effort=80 velocity=10
- joint LH_HAA: limit lower=-0.7853981633974483 upper=0.7853981633974483 effort=35 velocity=10 -> lower=-0.7853981633974483 upper=0.7853981633974483 effort=40 velocity=10
- joint LH_HFE: limit lower=-2.5 upper=1.57 effort=35 velocity=10 -> lower=-2.5 upper=1.57 effort=40 velocity=10
- joint LH_KFE: limit lower=-1.17453292519943295 upper=3.141592653589793 effort=45 velocity=10 -> lower=-1.17453292519943295 upper=3.141592653589793 effort=80 velocity=10
- joint RF_HAA: limit lower=-0.7853981633974483 upper=0.7853981633974483 effort=35 velocity=10 -> lower=-0.7853981633974483 upper=0.7853981633974483 effort=40 velocity=10
- joint RF_HFE: limit lower=-1.57 upper=2.5 effort=35 velocity=10 -> lower=-1.57 upper=2.5 effort=40 velocity=10
- joint RF_KFE: limit lower=-3.141592653589793 upper=1.17453292519943295 effort=45 velocity=10 -> lower=-3.141592653589793 upper=1.17453292519943295 effort=80 velocity=10
- joint RH_HAA: limit lower=-0.7853981633974483 upper=0.7853981633974483 effort=35 velocity=10 -> lower=-0.7853981633974483 upper=0.7853981633974483 effort=40 velocity=10
- joint RH_HFE: limit lower=-2.5 upper=1.57 effort=35 velocity=10 -> lower=-2.5 upper=1.57 effort=40 velocity=10
- joint RH_KFE: limit lower=-1.17453292519943295 upper=3.141592653589793 effort=45 velocity=10 -> lower=-1.17453292519943295 upper=3.141592653589793 effort=80 velocity=10

Commit message: update urdf

File: legged_gym/resources/robots/sirius/urdf/sirius_diff.urdf (robot description, URDF)
Before this commit: robot robot, 18 links, 17 joints
Joints:
- joint LF_HAA: limit lower=-0.7853981633974483 upper=0.7853981633974483 effort=40 velocity=10 -> lower=-0.7853981633974483 upper=0.7853981633974483 effort=35 velocity=10
- joint LF_HFE: limit lower=-1.57 upper=2.5 effort=40 velocity=10 -> lower=-1.57 upper=2.5 effort=35 velocity=10
- joint LF_KFE: limit lower=-3.141592653589793 upper=1.17453292519943295 effort=80 velocity=10 -> lower=-3.141592653589793 upper=1.17453292519943295 effort=70 velocity=8
- joint LH_HAA: limit lower=-0.7853981633974483 upper=0.7853981633974483 effort=40 velocity=10 -> lower=-0.7853981633974483 upper=0.7853981633974483 effort=35 velocity=10
- joint LH_HFE: limit lower=-2.5 upper=1.57 effort=40 velocity=10 -> lower=-2.5 upper=1.57 effort=35 velocity=10
- joint LH_KFE: limit lower=-1.17453292519943295 upper=3.141592653589793 effort=80 velocity=10 -> lower=-1.17453292519943295 upper=3.141592653589793 effort=70 velocity=8
- joint RF_HAA: limit lower=-0.7853981633974483 upper=0.7853981633974483 effort=40 velocity=10 -> lower=-0.7853981633974483 upper=0.7853981633974483 effort=35 velocity=10
- joint RF_HFE: limit lower=-1.57 upper=2.5 effort=40 velocity=10 -> lower=-1.57 upper=2.5 effort=35 velocity=10
- joint RF_KFE: limit lower=-3.141592653589793 upper=1.17453292519943295 effort=80 velocity=10 -> lower=-3.141592653589793 upper=1.17453292519943295 effort=70 velocity=8
- joint RH_HAA: limit lower=-0.7853981633974483 upper=0.7853981633974483 effort=40 velocity=10 -> lower=-0.7853981633974483 upper=0.7853981633974483 effort=35 velocity=10
- joint RH_HFE: limit lower=-2.5 upper=1.57 effort=40 velocity=10 -> lower=-2.5 upper=1.57 effort=35 velocity=10
- joint RH_KFE: limit lower=-1.17453292519943295 upper=3.141592653589793 effort=80 velocity=10 -> lower=-1.17453292519943295 upper=3.141592653589793 effort=70 velocity=8

Commit message: add fix action std adn new urdf

File: legged_gym/resources/robots/sirius/urdf/sirius_diff.urdf (robot description, URDF)
Before this commit: robot robot, 18 links, 17 joints
Joints:
- joint LF_HAA: limit lower=-0.7853981633974483 upper=0.7853981633974483 effort=35 velocity=10 -> lower=-0.7853981633974483 upper=0.7853981633974483 effort=35 velocity=18
- joint LF_HFE: limit lower=-1.57 upper=2.5 effort=35 velocity=10 -> lower=-1.57 upper=2.5 effort=35 velocity=18
- joint LF_KFE: limit lower=-3.141592653589793 upper=1.17453292519943295 effort=70 velocity=8 -> lower=-3.141592653589793 upper=1.17453292519943295 effort=70 velocity=10
- joint LH_HAA: limit lower=-0.7853981633974483 upper=0.7853981633974483 effort=35 velocity=10 -> lower=-0.7853981633974483 upper=0.7853981633974483 effort=35 velocity=18
- joint LH_HFE: limit lower=-2.5 upper=1.57 effort=35 velocity=10 -> lower=-2.5 upper=1.57 effort=35 velocity=18
- joint LH_KFE: limit lower=-1.17453292519943295 upper=3.141592653589793 effort=70 velocity=8 -> lower=-1.17453292519943295 upper=3.141592653589793 effort=70 velocity=10
- joint RF_HAA: limit lower=-0.7853981633974483 upper=0.7853981633974483 effort=35 velocity=10 -> lower=-0.7853981633974483 upper=0.7853981633974483 effort=35 velocity=18
- joint RF_HFE: limit lower=-1.57 upper=2.5 effort=35 velocity=10 -> lower=-1.57 upper=2.5 effort=35 velocity=18
- joint RF_KFE: limit lower=-3.141592653589793 upper=1.17453292519943295 effort=70 velocity=8 -> lower=-3.141592653589793 upper=1.17453292519943295 effort=70 velocity=10
- joint RH_HAA: limit lower=-0.7853981633974483 upper=0.7853981633974483 effort=35 velocity=10 -> lower=-0.7853981633974483 upper=0.7853981633974483 effort=35 velocity=18
- joint RH_HFE: limit lower=-2.5 upper=1.57 effort=35 velocity=10 -> lower=-2.5 upper=1.57 effort=35 velocity=18
- joint RH_KFE: limit lower=-1.17453292519943295 upper=3.141592653589793 effort=70 velocity=8 -> lower=-1.17453292519943295 upper=3.141592653589793 effort=70 velocity=10
